File: PCB/USBHume2.sch (EAGLE design)
At the start: 23 parts, among them IC1 LM1117MP-3.3

Commit message: Parts sizes fixed. Board errors fixed.
Parts:
- C1, C2, C3, C4, C6: device rcl:C-EUC0805 -> rcl:C-EUC1206K
- C5, C7: device rcl:CPOL-EUA/3216-18W -> rcl:CPOL-EUC/6032-28R
Changed lines of the file:
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@@
 <part name="X1" library="con-usb-3" deviceset="USB" device="-A-H"/>
 <part name="U1" library="RHT03_DHT-22_AM2302" deviceset="RHT03_DHT-22_AM2302" device="WIRED"/>
-<part name="C6" library="rcl" deviceset="C-EU" device="C0805" value="100n"/>
+<part name="C6" library="rcl" deviceset="C-EU" device="C1206K" value="100n"/>
 <part name="GND7" library="supply1" deviceset="GND" device=""/>
 <part name="STM32" library="stm32f0" deviceset="STM32F042" device=""/>
-<part name="C1" library="rcl" deviceset="C-EU" device="C0805" value="100n"/>
+<part name="C1" library="rcl" deviceset="C-EU" device="C1206K" value="100n"/>
 <part name="GND1" library="supply1" deviceset="GND" device=""/>
 <part name="+3V1" library="supply1" deviceset="+3V3" device=""/>
@@
 <part name="R4" library="rcl" deviceset="R-EU_" device="M0805" value="1k"/>
 <part name="LED3" library="led" deviceset="LED" device="CHIPLED_0805" value="ACT"/>
-<part name="C2" library="rcl" deviceset="C-EU" device="C0805" value="100n"/>
+<part name="C2" library="rcl" deviceset="C-EU" device="C1206K" value="100n"/>
 <part name="GND5" library="supply1" deviceset="GND" device=""/>
 <part name="JP3" library="pinhead" deviceset="PINHD-1X1" device="" value="NRST"/>
@@
 <part name="+3V5" library="supply1" deviceset="+3V3" device=""/>
 <part name="GND8" library="supply1" deviceset="GND" device=""/>
-<part name="C3" library="rcl" deviceset="C-EU" device="C0805" value="100n"/>
-<part name="C4" library="rcl" deviceset="C-EU" device="C0805" value="100n"/>
+<part name="C3" library="rcl" deviceset="C-EU" device="C1206K" value="100n"/>
+<part name="C4" library="rcl" deviceset="C-EU" device="C1206K" value="100n"/>
 <part name="GND9" library="supply1" deviceset="GND" device=""/>
 <part name="GND10" library="supply1" deviceset="GND" device=""/>
-<part name="C5" library="rcl" deviceset="CPOL-EU" device="A/3216-18W" value="10u"/>
-<part name="C7" library="rcl" deviceset="CPOL-EU" device="A/3216-18W" value="10u"/>
+<part name="C5" library="rcl" deviceset="CPOL-EU" device="C/6032-28R" value="10u"/>
+<part name="C7" library="rcl" deviceset="CPOL-EU" device="C/6032-28R" value="10u"/>
 <part name="GND11" library="supply1" deviceset="GND" device=""/>
 <part name="GND12" library="supply1" deviceset="GND" device=""/>

Commit message: Board simplification
Parts:
- removed JP3: NRST, pinhead:PINHD-1X1
- removed R5, R7: 33, rcl:R-EU_M0805
- removed R8: 1k5, rcl:R-EU_M0805
Connections:
- removed net N$16: R7.1, X1.D-
- removed net N$17: R5.1, R8.1, X1.D+
- net +3V3: no longer R8.2
- net N$15: no longer JP3.1
- net N$3: now also X1.D-; no longer R7.2
- net N$5: now also X1.D+; no longer R5.2
Changed lines of the file:
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@@
 <part name="C2" library="rcl" deviceset="C-EU" device="C1206K" value="100n"/>
 <part name="GND5" library="supply1" deviceset="GND" device=""/>
-<part name="JP3" library="pinhead" deviceset="PINHD-1X1" device="" value="NRST"/>
 <part name="JP4" library="pinhead" deviceset="PINHD-1X1" device="" value="3V3"/>
 <part name="JP5" library="pinhead" deviceset="PINHD-1X1" device="" value="GND"/>
@@
 <part name="GND11" library="supply1" deviceset="GND" device=""/>
 <part name="GND12" library="supply1" deviceset="GND" device=""/>
-<part name="R5" library="rcl" deviceset="R-EU_" device="M0805" value="33"/>
-<part name="R7" library="rcl" deviceset="R-EU_" device="M0805" value="33"/>
-<part name="R8" library="rcl" deviceset="R-EU_" device="M0805" value="1k5"/>
-<part name="+3V6" library="supply1" deviceset="+3V3" device=""/>
 </parts>
 <sheets>
@@
 <instance part="C2" gate="G$1" x="-53.34" y="7.62"/>
 <instance part="GND5" gate="1" x="-53.34" y="-5.08"/>
-<instance part="JP3" gate="G$1" x="-71.12" y="15.24" rot="R180"/>
 <instance part="JP4" gate="G$1" x="-63.5" y="71.12"/>
 <instance part="JP5" gate="G$1" x="-63.5" y="60.96"/>
@@
 <instance part="GND11" gate="1" x="-20.32" y="66.04"/>
 <instance part="GND12" gate="1" x="55.88" y="66.04"/>
-<instance part="R5" gate="G$1" x="162.56" y="5.08" rot="R180"/>
-<instance part="R7" gate="G$1" x="172.72" y="2.54" rot="R180"/>
-<instance part="R8" gate="G$1" x="180.34" y="12.7" rot="R90"/>
-<instance part="+3V6" gate="G$1" x="180.34" y="38.1"/>
 </instances>
 <busses>
@@
 <wire x1="63.5" y1="15.24" x2="127" y2="15.24" width="0.1524" layer="91"/>
 <wire x1="127" y1="15.24" x2="127" y2="2.54" width="0.1524" layer="91"/>
-<pinref part="R7" gate="G$1" pin="2"/>
-<wire x1="167.64" y1="2.54" x2="127" y2="2.54" width="0.1524" layer="91"/>
+<wire x1="198.12" y1="2.54" x2="127" y2="2.54" width="0.1524" layer="91"/>
+<pinref part="X1" gate="G$1" pin="D-"/>
 </segment>
 </net>
@@
 <pinref part="STM32" gate="G$1" pin="PA10[PA12]/USART1_RX/TIM1_CH3"/>
 <wire x1="124.46" y1="12.7" x2="63.5" y2="12.7" width="0.1524" layer="91"/>
-<pinref part="R5" gate="G$1" pin="2"/>
-<wire x1="157.48" y1="5.08" x2="124.46" y2="5.08" width="0.1524" layer="91"/>
+<wire x1="198.12" y1="5.08" x2="124.46" y2="5.08" width="0.1524" layer="91"/>
+<pinref part="X1" gate="G$1" pin="D+"/>
 </segment>
 </net>
@@
 <junction x="55.88" y="86.36"/>
 </segment>
-<segment>
-<pinref part="R8" gate="G$1" pin="2"/>
-<pinref part="+3V6" gate="G$1" pin="+3V3"/>
-<wire x1="180.34" y1="17.78" x2="180.34" y2="35.56" width="0.1524" layer="91"/>
-</segment>
 </net>
 <net name="N$7" class="0">
@@
 <wire x1="-30.48" y1="15.24" x2="-53.34" y2="15.24" width="0.1524" layer="91"/>
 <wire x1="-53.34" y1="15.24" x2="-53.34" y2="10.16" width="0.1524" layer="91"/>
-<pinref part="JP3" gate="G$1" pin="1"/>
-<wire x1="-53.34" y1="15.24" x2="-68.58" y2="15.24" width="0.1524" layer="91"/>
-<junction x="-53.34" y="15.24"/>
-</segment>
-</net>
-<net name="N$16" class="0">
-<segment>
-<pinref part="X1" gate="G$1" pin="D-"/>
-<pinref part="R7" gate="G$1" pin="1"/>
-<wire x1="198.12" y1="2.54" x2="177.8" y2="2.54" width="0.1524" layer="91"/>
-</segment>
-</net>
-<net name="N$17" class="0">
-<segment>
-<pinref part="R5" gate="G$1" pin="1"/>
-<pinref part="X1" gate="G$1" pin="D+"/>
-<wire x1="167.64" y1="5.08" x2="180.34" y2="5.08" width="0.1524" layer="91"/>
-<pinref part="R8" gate="G$1" pin="1"/>
-<wire x1="180.34" y1="5.08" x2="198.12" y2="5.08" width="0.1524" layer="91"/>
-<wire x1="180.34" y1="5.08" x2="180.34" y2="7.62" width="0.1524" layer="91"/>
-<junction x="180.34" y="5.08"/>
-</segment>
-</net>
+</segment>
+</net>

Commit message: Programming pins grouped
Parts:
- removed JP2: SWDCLK, pinhead:PINHD-1X1
- removed JP4: 3V3, pinhead:PINHD-1X1
- removed JP5: GND, pinhead:PINHD-1X1
- added JP3: (no value), pinhead:PINHD-1X2
- JP1: value SWDIO -> (none); device pinhead:PINHD-1X1 -> pinhead:PINHD-1X2
Connections:
- net +3V3: now also JP1.1; no longer JP4.1
- net GND: now also JP1.2; no longer JP5.1
- net N$10: now also JP3.2; no longer JP2.1
- net N$9: now also JP3.1; no longer JP1.1
Changed lines of the file:
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@@
 <part name="GND3" library="supply1" deviceset="GND" device=""/>
 <part name="R1" library="rcl" deviceset="R-EU_" device="M0805" value="510"/>
-<part name="JP1" library="pinhead" deviceset="PINHD-1X1" device="" value="SWDIO"/>
-<part name="JP2" library="pinhead" deviceset="PINHD-1X1" device="" value="SWDCLK"/>
 <part name="GND4" library="supply1" deviceset="GND" device=""/>
 <part name="R4" library="rcl" deviceset="R-EU_" device="M0805" value="1k"/>
@@
 <part name="C2" library="rcl" deviceset="C-EU" device="C1206K" value="100n"/>
 <part name="GND5" library="supply1" deviceset="GND" device=""/>
-<part name="JP4" library="pinhead" deviceset="PINHD-1X1" device="" value="3V3"/>
-<part name="JP5" library="pinhead" deviceset="PINHD-1X1" device="" value="GND"/>
 <part name="+3V2" library="supply1" deviceset="+3V3" device=""/>
 <part name="GND6" library="supply1" deviceset="GND" device=""/>
@@
 <part name="GND11" library="supply1" deviceset="GND" device=""/>
 <part name="GND12" library="supply1" deviceset="GND" device=""/>
+<part name="JP3" library="pinhead" deviceset="PINHD-1X2" device=""/>
+<part name="JP1" library="pinhead" deviceset="PINHD-1X2" device=""/>
 </parts>
 <sheets>
@@
 <instance part="GND3" gate="1" x="-40.64" y="-5.08"/>
 <instance part="R1" gate="G$1" x="-40.64" y="5.08" rot="R90"/>
-<instance part="JP1" gate="G$1" x="114.3" y="-5.08"/>
-<instance part="JP2" gate="G$1" x="114.3" y="-17.78"/>
 <instance part="GND4" gate="1" x="109.22" y="7.62"/>
 <instance part="R4" gate="G$1" x="73.66" y="25.4" rot="R180"/>
@@
 <instance part="C2" gate="G$1" x="-53.34" y="7.62"/>
 <instance part="GND5" gate="1" x="-53.34" y="-5.08"/>
-<instance part="JP4" gate="G$1" x="-63.5" y="71.12"/>
-<instance part="JP5" gate="G$1" x="-63.5" y="60.96"/>
 <instance part="+3V2" gate="G$1" x="-76.2" y="81.28"/>
 <instance part="GND6" gate="1" x="-76.2" y="53.34"/>
@@
 <instance part="GND11" gate="1" x="-20.32" y="66.04"/>
 <instance part="GND12" gate="1" x="55.88" y="66.04"/>
+<instance part="JP3" gate="G$1" x="132.08" y="-12.7"/>
+<instance part="JP1" gate="G$1" x="-55.88" y="63.5"/>
 </instances>
 <busses>
@@
 </segment>
 <segment>
-<pinref part="JP5" gate="G$1" pin="1"/>
 <pinref part="GND6" gate="1" pin="GND"/>
-<wire x1="-66.04" y1="60.96" x2="-76.2" y2="60.96" width="0.1524" layer="91"/>
-<wire x1="-76.2" y1="60.96" x2="-76.2" y2="55.88" width="0.1524" layer="91"/>
+<wire x1="-76.2" y1="63.5" x2="-76.2" y2="55.88" width="0.1524" layer="91"/>
+<pinref part="JP1" gate="G$1" pin="2"/>
+<wire x1="-58.42" y1="63.5" x2="-76.2" y2="63.5" width="0.1524" layer="91"/>
 </segment>
 <segment>
@@
 </segment>
 <segment>
-<pinref part="JP4" gate="G$1" pin="1"/>
 <pinref part="+3V2" gate="G$1" pin="+3V3"/>
-<wire x1="-66.04" y1="71.12" x2="-76.2" y2="71.12" width="0.1524" layer="91"/>
-<wire x1="-76.2" y1="71.12" x2="-76.2" y2="78.74" width="0.1524" layer="91"/>
+<wire x1="-76.2" y1="66.04" x2="-76.2" y2="78.74" width="0.1524" layer="91"/>
+<pinref part="JP1" gate="G$1" pin="1"/>
+<wire x1="-58.42" y1="66.04" x2="-76.2" y2="66.04" width="0.1524" layer="91"/>
 </segment>
 <segment>
@@
 <pinref part="STM32" gate="G$1" pin="PA13/SWDIO"/>
 <wire x1="63.5" y1="10.16" x2="99.06" y2="10.16" width="0.1524" layer="91"/>
-<wire x1="99.06" y1="10.16" x2="99.06" y2="-5.08" width="0.1524" layer="91"/>
-<pinref part="JP1" gate="G$1" pin="1"/>
-<wire x1="99.06" y1="-5.08" x2="111.76" y2="-5.08" width="0.1524" layer="91"/>
+<wire x1="99.06" y1="10.16" x2="99.06" y2="-10.16" width="0.1524" layer="91"/>
+<pinref part="JP3" gate="G$1" pin="1"/>
+<wire x1="129.54" y1="-10.16" x2="99.06" y2="-10.16" width="0.1524" layer="91"/>
 </segment>
 </net>
 <net name="N$10" class="0">
 <segment>
-<pinref part="JP2" gate="G$1" pin="1"/>
-<wire x1="111.76" y1="-17.78" x2="96.52" y2="-17.78" width="0.1524" layer="91"/>
-<wire x1="96.52" y1="-17.78" x2="96.52" y2="7.62" width="0.1524" layer="91"/>
 <pinref part="STM32" gate="G$1" pin="PA14/USART2_TX/SWCLK"/>
+<wire x1="96.52" y1="-12.7" x2="96.52" y2="7.62" width="0.1524" layer="91"/>
 <wire x1="96.52" y1="7.62" x2="63.5" y2="7.62" width="0.1524" layer="91"/>
-</segment>
-</net>
+<pinref part="JP3" gate="G$1" pin="2"/>
+<wire x1="129.54" y1="-12.7" x2="96.52" y2="-12.7" width="0.1524" layer="91"/>
+</segment>
+</net>
